Commit message: URDF cleanup and launchfile tweaks

File: src/description/tuppy_description.urdf (robot description, URDF)
Before this commit: robot tuppy_description, 10 links, 9 joints
Links:
- removed link bottom_frame
- added link back_frame; visual box size=${frame_x} ${frame_y} ${frame_z}
- added link lidar; visual cylinder length=${lidar_l} radius=${lidar_r}
- added link sensor_holder; visual box size=${frame_x} ${frame_y} ${frame_z}
- link base_link: geometry 
- link camera: geometry visual box size=${camera_x} ${camera_y} ${camera_z}
- link front_frame: geometry visual box size=${frame_x} ${frame_y} ${frame_z}
- link left_hull: geometry visual box size=${hull_x} ${hull_y} ${hull_z}
- link middle_frame: geometry visual box size=${frame_x} ${frame_y} ${frame_z}
- link polycarbsheet: geometry visual box size=${polycarb_x} ${polycarb_y} ${polycarb_z}
- link right_hull: geometry visual box size=${hull_x} ${hull_y} ${hull_z}
- link tupperware: geometry visual box size=${tuppy_x} ${tuppy_y} ${tuppy_z}
Joints:
- removed joint baselink_frontframe
- removed joint frontframe_camear
- removed joint frontframe_lefthull
- removed joint frontframe_middleframe
- removed joint lefthull_righthull
- removed joint middleframe_bottomframe
- removed joint middleframe_polycarb
- removed joint polycarb_tupperware
- added joint base_tuppy: type fixed, parent base_link, child tupperware, origin xyz=0 0 0 rpy=0 0 0
- added joint holder_camera: type fixed, parent sensor_holder, child camera, origin xyz=0 0 0 rpy=0 0 0
- added joint holder_lidar: type fixed, parent sensor_holder, child lidar, origin xyz=0 0 ${lidar_l/2} rpy=0 0 0
- added joint lefthull_holder: type fixed, parent front_frame, child sensor_holder, origin xyz=0 0 ${polycarb_z+frame_z/2} rpy=0 0 0
- added joint middlef_lefthull: type fixed, parent middle_frame, child left_hull, origin xyz=${hull_x/2-polycarb_x/2} ${polycarb_y/2-hull_y/2} ${-(hull_z/2+frame_z/2)} rpy=0 0 0
- added joint middlef_righthull: type fixed, parent middle_frame, child right_hull, origin xyz=${hull_x/2-polycarb_x/2} ${-(polycarb_y/2-hull_y/2)} ${-(hull_z/2+frame_z/2)} rpy=0 0 0
- added joint polyf_back: type fixed, parent polycarbsheet, child back_frame, origin xyz=${-(polycarb_x/2-frame_z/2)} 0 ${-frame_z/2+polycarb_z/2}} rpy=0 0 0
- added joint polyf_front: type fixed, parent polycarbsheet, child front_frame, origin xyz=${polycarb_x/2-frame_z/2} 0 ${-frame_z/2+polycarb_z/2} rpy=0 0 0
- added joint polyf_middle: type fixed, parent polycarbsheet, child middle_frame, origin xyz=0 0 ${-frame_z/2+polycarb_z/2}} rpy=0 0 0
- added joint tuppy_poly: type fixed, parent tupperware, child polycarbsheet, origin xyz=0 0 ${-(frame_z/2+tuppy_z/2)} rpy=0 0 0
- joint base_joint: origin xyz=0.0 0.0 -0.18 rpy=0 0 0 -> xyz=0 0 ${-(tuppy_z/2+polycarb_z+frame_z+hull_z)} rpy=0 0 0
